Commit message: Added Gym implementation for lift cube (not functional)

File: gym_drake_lca/low-cost-arm.urdf (robot description, URDF)
Before this commit: robot low-cost-arm, 7 links, 6 joints
Links:
- removed link elbow-to-wrist-motor-reference_v1_1
- removed link first-bracket-motor_1
- removed link gripper-moving-part-dumb_v2_1
- removed link gripper-static-motor_v2_1
- removed link shoulder-to-elbow-motor_v1_1
- added link elbow, mass 0.05261369068977079; collision mesh filename=assets/shoulder-to-elbow-motor_v1_1.obj scale=0.001 0.001 0.001; visual mesh filename=assets/shoulder-to-elbow-motor_v1_1.obj scale=0.001 0.001 0.001
- added link gripper_moving_part, mass 0.013583445641331692; collision mesh filename=assets/gripper-moving-part-dumb_v2_1.obj scale=0.001 0.001 0.001; visual mesh filename=assets/gripper-moving-part-dumb_v2_1.obj scale=0.001 0.001 0.001
- added link gripper_static_part, mass 0.030801959916802346; collision mesh filename=assets/gripper-static-motor_v2_1.obj scale=0.001 0.001 0.001; visual mesh filename=assets/gripper-static-motor_v2_1.obj scale=0.001 0.001 0.001
- added link shoulder, mass 0.050669759178187244; collision mesh filename=assets/first-bracket-motor_1.obj scale=0.001 0.001 0.001; visual mesh filename=assets/first-bracket-motor_1.obj scale=0.001 0.001 0.001
- added link wrist, mass 0.02059907441055582; collision mesh filename=assets/elbow-to-wrist-motor-reference_v1_1.obj scale=0.001 0.001 0.001; visual mesh filename=assets/elbow-to-wrist-motor-reference_v1_1.obj scale=0.001 0.001 0.001
Joints:
- joint joint_2: child first-bracket-motor_1 -> shoulder
- joint joint_3: child shoulder-to-elbow-motor_v1_1 -> elbow; parent first-bracket-motor_1 -> shoulder
- joint joint_5: child elbow-to-wrist-motor-reference_v1_1 -> wrist; parent shoulder-to-elbow-motor_v1_1 -> elbow
- joint joint_6: child gripper-static-motor_v2_1 -> gripper_static_part; parent elbow-to-wrist-motor-reference_v1_1 -> wrist
- joint joint_7: child gripper-moving-part-dumb_v2_1 -> gripper_moving_part; parent gripper-static-motor_v2_1 -> gripper_static_part
